Commit message: added mass_sensor, gif_record

File: custom_envs/heavy-pb/heavy_pb/resources/forwarder/Forwarder.urdf (robot description, URDF)
Before this commit: robot Forwarder, 9 links, 8 joints
Links:
- added link extension_arm1, mass 385.82757219552406; collision mesh filename=meshes/extension_arm1.stl scale=0.001 0.001 0.001; visual mesh filename=meshes/extension_arm1.stl scale=0.001 0.001 0.001
- link base_link: mass 25822.657136799415 -> 25822.65720552091
- link extension1: mass 422.2365549320586 -> 250.5548388854696
Joints:
- removed joint Revolute_24
- removed joint Revolute_27
- added joint Revolute_36: type continuous, parent craneArm1, child extension_arm1, origin xyz=0.22 2.647071 2.090045 rpy=0 0 0, axis 1.0 -0.0 0.0, limit lower=-1.54 upper=0.43
- added joint Revolute_38: type continuous, parent extension1, child intermediateHookJnt1, origin xyz=-0.03 1.91394 -0.132446 rpy=0 0 0, axis 1.0 -0.0 0.0
- added joint Slider_37: type prismatic, parent extension_arm1, child extension1, origin xyz=-0.14 1.539638 -0.097247 rpy=0 0 0, axis -0.0 -0.991429 0.130644, limit lower=-.8 upper=1
- joint Revolute_1: limit lower=-1.54 upper=1.54 -> lower=-1.04 upper=1.04
- joint Revolute_16: axis -0.0 -1.0 0.000365 -> -0.0 -0.984744 0.174008; origin xyz=-0.06 0.039916 -0.232475 rpy=0 0 0 -> xyz=0.06 -0.001061 -0.235875 rpy=0 0 0
- joint Revolute_25: limit lower=-1.54 upper=0.60 -> lower=-0.43 upper=0.33
- joint Revolute_26: axis 0.0 -0.000365 -1.0 -> 0.0 -0.174008 -0.984744; limit lower=-3.14 upper=3.14 -> lower=0 upper=1.54; origin xyz=0.0 -0.040079 -0.214985 rpy=0 0 0 -> xyz=0.0 -0.076801 -0.204759 rpy=0 0 0
- joint Revolute_30: axis -0.0 -1.0 0.000365 -> -0.0 -0.984744 0.174008; limit (none) -> lower=-.6 upper=.6; origin xyz=0.28 0.149937 -0.173825 rpy=0 0 0 -> xyz=0.28 0.117474 -0.19722 rpy=0 0 0
- joint Revolute_31: axis -0.0 -1.0 0.000365 -> -0.0 -0.984744 0.174008; limit lower=-1.54 upper=.6 -> lower=-.6 upper=.6; origin xyz=-0.28 0.149937 -0.173825 rpy=0 0 0 -> xyz=-0.28 0.117474 -0.19722 rpy=0 0 0

Commit message: new_actuations_tests

File: custom_envs/heavy-pb/heavy_pb/resources/forwarder/Forwarder.urdf (robot description, URDF)
Before this commit: robot Forwarder, 10 links, 9 joints
Joints:
- joint Revolute_1: limit lower=-1.04 upper=1.04 -> lower=-1.54 upper=1.54

Commit message: added feature extractor

File: custom_envs/heavy-pb/heavy_pb/resources/forwarder/Forwarder.urdf (robot description, URDF)
Before this commit: robot Forwarder, 10 links, 9 joints
Joints:
- joint Revolute_16: limit (none) -> lower=-.3 upper=.3 effort=1 velocity=5; type continuous -> revolute
- joint Revolute_38: limit (none) -> lower=-.8 upper=.8 effort=1 velocity=5; type continuous -> revolute

Commit message: removed pos check from frameskip

File: custom_envs/heavy-pb/heavy_pb/resources/forwarder/Forwarder.urdf (robot description, URDF)
Before this commit: robot Forwarder, 10 links, 9 joints
Joints:
- joint Revolute_26: type continuous -> revolute

Commit message: changed camera pos

File: custom_envs/heavy-pb/heavy_pb/resources/forwarder/Forwarder.urdf (robot description, URDF)
Before this commit: robot Forwarder, 10 links, 9 joints
Joints:
- joint Revolute_26: limit lower=0 upper=1.54 -> lower=0 upper=2
